Commit message: ⚡️ perf(arm): 放宽关节速度规划上限并补充 MoveIt 加速度限制
1. URDF 关节速度限制从 1.57 提升至固件规格 (J1-J4: 3.1416, J5-J6: 3.4907 rad/s)
2. launch 增加 robot_description_planning joint_limits (max_acceleration 5.0 rad/s²)
   URDF 不含加速度限制，缺失时 TOTG 时间参数化按默认 1.0 rad/s² 规划导致移动慢

File: src/elfin_description/urdf/elfin5.urdf.xacro (robot description, xacro)
@@ -66,5 +66,5 @@
     <child link="elfin_link1" />
     <axis xyz="0 0 1" />
-    <limit lower="-3.14" upper="3.14" effort="420" velocity="1.57" />
+    <limit lower="-3.14" upper="3.14" effort="420" velocity="3.1416" />
   </joint>
   <link name="elfin_link2">
@@ -96,5 +96,5 @@
     <child link="elfin_link2" />
     <axis xyz="0 0 1" />
-    <limit lower="-2.35" upper="2.35" effort="420" velocity="1.57" />
+    <limit lower="-2.35" upper="2.35" effort="420" velocity="3.1416" />
   </joint>
   <link name="elfin_link3">
@@ -126,5 +126,5 @@
     <child link="elfin_link3" />
     <axis xyz="0 0 1" />
-    <limit lower="-2.61" upper="2.61" effort="200" velocity="1.57" />
+    <limit lower="-2.61" upper="2.61" effort="200" velocity="3.1416" />
   </joint>
   <link name="elfin_link4">
@@ -156,5 +156,5 @@
     <child link="elfin_link4" />
     <axis xyz="0 0 1" />
-    <limit lower="-3.14" upper="3.14" effort="200" velocity="1.57" />
+    <limit lower="-3.14" upper="3.14" effort="200" velocity="3.1416" />
   </joint>
   <link name="elfin_link5">
@@ -186,5 +186,5 @@
     <child link="elfin_link5" />
     <axis xyz="0 0 1" />
-    <limit lower="-2.56" upper="2.56" effort="69" velocity="1.57" />
+    <limit lower="-2.56" upper="2.56" effort="69" velocity="3.4907" />
   </joint>
   <link name="elfin_link6">
@@ -216,5 +216,5 @@
     <child link="elfin_link6" />
     <axis xyz="0 0 1" />
-    <limit lower="-3.14" upper="3.14" effort="69" velocity="1.57" />
+    <limit lower="-3.14" upper="3.14" effort="69" velocity="3.4907" />
   </joint>
   <link name="elfin_end_link"/>
